File: RHC12-BTA.sch (EAGLE design)
At the start: 6 parts

Commit message: Uh...
Parts:
- JP1, JP2, JP3: device SparkFun-Connectors:M04NO_SILK_ALL_ROUND -> SparkFun-Connectors:M04SMD
- R1, R2: device SparkFun-Passives:RESISTORPTH-1/4W -> SparkFun-Passives:RESISTOR0603-RES
Changed lines of the file:
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@@
 <?xml version="1.0" encoding="utf-8"?>
 <!DOCTYPE eagle SYSTEM "eagle.dtd">
-<eagle version="7.5.0">
+<eagle version="7.2.0">
 <drawing>
 <settings>
@@
 <parts>
 <part name="JP5" library="SparkFun-Connectors" deviceset="M06" device="VERNIER-ANALOG" value="BTA"/>
-<part name="JP1" library="SparkFun-Connectors" deviceset="M04" device="NO_SILK_ALL_ROUND"/>
-<part name="JP2" library="SparkFun-Connectors" deviceset="M04" device="NO_SILK_ALL_ROUND"/>
-<part name="JP3" library="SparkFun-Connectors" deviceset="M04" device="NO_SILK_ALL_ROUND"/>
-<part name="R1" library="SparkFun-Passives" deviceset="RESISTOR" device="PTH-1/4W"/>
-<part name="R2" library="SparkFun-Passives" deviceset="RESISTOR" device="PTH-1/4W"/>
+<part name="JP1" library="SparkFun-Connectors" deviceset="M04" device="SMD"/>
+<part name="JP2" library="SparkFun-Connectors" deviceset="M04" device="SMD"/>
+<part name="JP3" library="SparkFun-Connectors" deviceset="M04" device="SMD"/>
+<part name="R1" library="SparkFun-Passives" deviceset="RESISTOR" device="0603-RES"/>
+<part name="R2" library="SparkFun-Passives" deviceset="RESISTOR" device="0603-RES"/>
 </parts>
 <sheets>
